File: workshop_controller.sch (KiCad schematic (older format))
At the start: 2 parts

Commit message: Add a few components
Parts:
- added BT?: Battery, symbol Device:Battery
- added J3: AudioJack3, symbol Connector:AudioJack3
- added J4: Micro_SD_Card_Det, symbol Connector:Micro_SD_Card_Det
- added LS1: Speaker, symbol Device:Speaker
- added MK1: Microphone, symbol Device:Microphone
- added RV1: R_POT_Dual, symbol Device:R_POT_Dual
- added SW1, SW2: SW_Push, symbol Switch:SW_Push
- added U1: MPU-9250, Sensor_Motion:InvenSense_QFN-24_3x3mm_P0.4mm, symbol Sensor_Motion:MPU-9250
- added U2: BME280, Package_LGA:Bosch_LGA-8_2.5x2.5mm_P0.65mm_ClockwisePinNumbering, symbol Sensor:BME280
- gave numbers to parts that had none: 2
Changed lines of the file:
@@
 EESchema Schematic File Version 4
 LIBS:workshop_controller-cache
-EELAYER 29 0
+EELAYER 26 0
 EELAYER END
 $Descr A4 11693 8268
@@
 $EndDescr
 $Comp
-L Connector_Generic:Conn_02x10_Odd_Even J?
+L Connector_Generic:Conn_02x10_Odd_Even J1
 U 1 1 5C5F462B
 P 4750 3300
-F 0 "J?" H 4800 3917 50  0000 C CNN
+F 0 "J1" H 4800 3917 50  0000 C CNN
 F 1 "Conn_02x10_Odd_Even" H 4800 3826 50  0000 C CNN
 F 2 "" H 4750 3300 50  0001 C CNN
@@
 $EndComp
 $Comp
-L Connector_Generic:Conn_02x10_Odd_Even J?
+L Connector_Generic:Conn_02x10_Odd_Even J2
 U 1 1 5C5F4734
 P 7000 3300
-F 0 "J?" H 7050 3917 50  0000 C CNN
+F 0 "J2" H 7050 3917 50  0000 C CNN
 F 1 "Conn_02x10_Odd_Even" H 7050 3826 50  0000 C CNN
 F 2 "" H 7000 3300 50  0001 C CNN
@@
 $EndComp
 $Comp
-L power:GND #PWR?
+L power:GND #PWR0101
 U 1 1 5C5F47BB
 P 4400 2900
-F 0 "#PWR?" H 4400 2650 50  0001 C CNN
+F 0 "#PWR0101" H 4400 2650 50  0001 C CNN
 F 1 "GND" V 4405 2772 50  0000 R CNN
 F 2 "" H 4400 2900 50  0001 C CNN
@@
 PIN_SD3
 $Comp
-L power:GND #PWR?
+L power:GND #PWR0102
 U 1 1 5C5F4AB8
 P 7450 2900
-F 0 "#PWR?" H 7450 2650 50  0001 C CNN
+F 0 "#PWR0102" H 7450 2650 50  0001 C CNN
 F 1 "GND" V 7455 2772 50  0000 R CNN
 F 2 "" H 7450 2900 50  0001 C CNN
@@
 PIN_16
 $Comp
-L power:GND #PWR?
+L power:GND #PWR0103
 U 1 1 5C5F4C3F
 P 6650 3500
-F 0 "#PWR?" H 6650 3250 50  0001 C CNN
+F 0 "#PWR0103" H 6650 3250 50  0001 C CNN
 F 1 "GND" V 6655 3372 50  0000 R CNN
 F 2 "" H 6650 3500 50  0001 C CNN
@@
 	4400 3800 4550 3800
 $Comp
-L power:+5V #PWR?
+L power:+5V #PWR0104
 U 1 1 5C5FB601
 P 6650 3600
-F 0 "#PWR?" H 6650 3450 50  0001 C CNN
+F 0 "#PWR0104" H 6650 3450 50  0001 C CNN
 F 1 "+5V" V 6665 3728 50  0000 L CNN
 F 2 "" H 6650 3600 50  0001 C CNN
@@
 	6650 3600 6800 3600
 $Comp
-L power:+3V3 #PWR?
+L power:+3V3 #PWR0105
 U 1 1 5C5FC146
 P 5200 3600
-F 0 "#PWR?" H 5200 3450 50  0001 C CNN
+F 0 "#PWR0105" H 5200 3450 50  0001 C CNN
 F 1 "+3V3" V 5215 3728 50  0000 L CNN
 F 2 "" H 5200 3600 50  0001 C CNN
@@
 Wire Wire Line
 	5200 2900 5050 2900
+$Comp
+L Sensor_Motion:MPU-9250 U1
+U 1 1 5CA64D58
+P 5900 5600
+F 0 "U1" H 5900 4614 50  0000 C CNN
+F 1 "MPU-9250" H 5900 4523 50  0000 C CNN
+F 2 "Sensor_Motion:InvenSense_QFN-24_3x3mm_P0.4mm" H 5900 4600 50  0001 C CNN
+F 3 "https://store.invensense.com/datasheets/invensense/MPU9250REV1.0.pdf" H 5900 5450 50  0001 C CNN
+	1    5900 5600
+	1    0    0    -1
+$EndComp
+$Comp
+L Sensor:BME280 U2
+U 1 1 5CA64E9A
+P 3850 5400
+F 0 "U2" H 3420 5446 50  0000 R CNN
+F 1 "BME280" H 3420 5355 50  0000 R CNN
+F 2 "Package_LGA:Bosch_LGA-8_2.5x2.5mm_P0.65mm_ClockwisePinNumbering" H 3850 5200 50  0001 C CNN
+F 3 "https://ae-bst.resource.bosch.com/media/_tech/media/datasheets/BST-BME280_DS001-11.pdf" H 3850 5200 50  0001 C CNN
+	1    3850 5400
+	1    0    0    -1
+$EndComp
+$Comp
+L Switch:SW_Push SW1
+U 1 1 5CA65465
+P 9150 1700
+F 0 "SW1" H 9150 1985 50  0000 C CNN
+F 1 "SW_Push" H 9150 1894 50  0000 C CNN
+F 2 "" H 9150 1900 50  0001 C CNN
+F 3 "" H 9150 1900 50  0001 C CNN
+	1    9150 1700
+	1    0    0    -1
+$EndComp
+$Comp
+L Switch:SW_Push SW2
+U 1 1 5CA6551B
+P 9150 2300
+F 0 "SW2" H 9150 2585 50  0000 C CNN
+F 1 "SW_Push" H 9150 2494 50  0000 C CNN
+F 2 "" H 9150 2500 50  0001 C CNN
+F 3 "" H 9150 2500 50  0001 C CNN
+	1    9150 2300
+	1    0    0    -1
+$EndComp
+$Comp
+L Connector:AudioJack3 J3
+U 1 1 5CA656CD
+P 2350 6300
+F 0 "J3" H 2330 6625 50  0000 C CNN
+F 1 "AudioJack3" H 2330 6534 50  0000 C CNN
+F 2 "" H 2350 6300 50  0001 C CNN
+F 3 "~" H 2350 6300 50  0001 C CNN
+	1    2350 6300
+	1    0    0    -1
+$EndComp
+$Comp
+L Device:R_POT_Dual RV1
+U 1 1 5CA65DAB
+P 2500 3800
+F 0 "RV1" H 2500 3568 50  0000 C CNN
+F 1 "R_POT_Dual" H 2500 3477 50  0000 C CNN
+F 2 "" H 2750 3725 50  0001 C CNN
+F 3 "~" H 2750 3725 50  0001 C CNN
+	1    2500 3800
+	1    0    0    -1
+$EndComp
+$Comp
+L Device:Speaker LS1
+U 1 1 5CA66A12
+P 5800 1650
+F 0 "LS1" H 5970 1646 50  0000 L CNN
+F 1 "Speaker" H 5970 1555 50  0000 L CNN
+F 2 "" H 5800 1450 50  0001 C CNN
+F 3 "~" H 5790 1600 50  0001 C CNN
+	1    5800 1650
+	1    0    0    -1
+$EndComp
+$Comp
+L Device:Microphone MK1
+U 1 1 5CA66C89
+P 4600 1700
+F 0 "MK1" H 4730 1746 50  0000 L CNN
+F 1 "Microphone" H 4730 1655 50  0000 L CNN
+F 2 "" V 4600 1800 50  0001 C CNN
+F 3 "~" V 4600 1800 50  0001 C CNN
+	1    4600 1700
+	1    0    0    -1
+$EndComp
+$Comp
+L Connector:Micro_SD_Card_Det J4
+U 1 1 5CA66F96
+P 8800 5150
+F 0 "J4" H 8750 5967 50  0000 C CNN
+F 1 "Micro_SD_Card_Det" H 8750 5876 50  0000 C CNN
+F 2 "" H 10850 5850 50  0001 C CNN
+F 3 "https://www.hirose.com/product/en/download_file/key_name/DM3/category/Catalog/doc_file_id/49662/?file_category_id=4&item_id=195&is_series=1" H 8800 5250 50  0001 C CNN
+	1    8800 5150
+	1    0    0    -1
+$EndComp
+$Comp
+L Device:Battery BT?
+U 1 1 5CA68FEC
+P 3100 2400
+F 0 "BT?" H 3208 2446 50  0000 L CNN
+F 1 "Battery" H 3208 2355 50  0000 L CNN
+F 2 "" V 3100 2460 50  0001 C CNN
+F 3 "~" V 3100 2460 50  0001 C CNN
+	1    3100 2400
+	1    0    0    -1
+$EndComp
 $EndSCHEMATC

Commit message: Add some footprints
Parts:
- removed BT?: Battery, symbol Device:Battery
- removed J4: Micro_SD_Card_Det, symbol Connector:Micro_SD_Card_Det
- added MICRO_SD1: Conn_01x06_Male, symbol Connector:Conn_01x06_Male
- added U3: MCP23S17_SS, Package_SO:SSOP-28_5.3x10.2mm_P0.65mm, symbol Interface_Expansion:MCP23S17_SS
- J1, J2: footprint (none) -> Connector_PinHeader_2.54mm:PinHeader_2x10_P2.54mm_Vertical
- renumbered RV1 to JOYSTICK_LEFT1
Connections:
- wire segments 38 -> 77
Other:
- moved on the sheet: J3, JOYSTICK_LEFT1, LS1, MK1, U1, U2

Commit message: Aesthetic changes
Parts:
- added SPI_HEADER: Conn_01x06_Female, symbol Connector:Conn_01x06_Female
Connections:
- net +3V3: now also SPI_HEADER.1 (Pin_1)
- net GND: now also SW1.1, SW2.1, SPI_HEADER.6 (Pin_6)
- net PIN_18: now also SPI_HEADER.4 (Pin_4); no longer U1.23 (SCL/SCLK), U2.4 (SCK)
- net PIN_19: now also SPI_HEADER.5 (Pin_5); no longer U1.9 (AD0/MISO), U2.3 (SDI)
- net PIN_23: now also SPI_HEADER.3 (Pin_3); no longer U1.24 (SDA/MOSI), U2.5 (SDO)
- net PIN_25: now also U1.24 (SDA/MOSI), U2.3 (SDI)
- net PIN_27: now also U1.23 (SCL/SCLK), U2.4 (SCK)
- net PIN_5: now also SW1.2
- net PIN_TMS: now also SW2.2
Other:
- moved on the sheet: SW1, SW2, U1, U2
Changed lines of the file:
@@
 	6650 2900 6800 2900
 Wire Wire Line
-	7450 3000 7300 3000
-Wire Wire Line
 	7450 3200 7300 3200
 Wire Wire Line
@@
 	5050 3700 5200 3700
 Wire Wire Line
-	5200 3500 5050 3500
-Wire Wire Line
 	4400 3200 4550 3200
 Wire Wire Line
@@
 Wire Wire Line
 	4550 3400 4400 3400
-Wire Wire Line
-	4400 3500 4550 3500
 Wire Wire Line
 	4550 3700 4400 3700
@@
 L Sensor_Motion:MPU-9250 U1
 U 1 1 5CA64D58
-P 6800 5650
-F 0 "U1" H 6800 4664 50  0000 C CNN
-F 1 "MPU-9250" H 6800 4573 50  0000 C CNN
-F 2 "Sensor_Motion:InvenSense_QFN-24_3x3mm_P0.4mm" H 6800 4650 50  0001 C CNN
-F 3 "https://store.invensense.com/datasheets/invensense/MPU9250REV1.0.pdf" H 6800 5500 50  0001 C CNN
-	1    6800 5650
+P 8700 5350
+F 0 "U1" H 8700 4364 50  0000 C CNN
+F 1 "MPU-9250" H 8700 4273 50  0000 C CNN
+F 2 "Sensor_Motion:InvenSense_QFN-24_3x3mm_P0.4mm" H 8700 4350 50  0001 C CNN
+F 3 "https://store.invensense.com/datasheets/invensense/MPU9250REV1.0.pdf" H 8700 5200 50  0001 C CNN
+	1    8700 5350
 	1    0    0    -1
 $EndComp
@@
 L Sensor:BME280 U2
 U 1 1 5CA64E9A
-P 4600 4800
-F 0 "U2" H 4170 4846 50  0000 R CNN
-F 1 "BME280" H 4170 4755 50  0000 R CNN
-F 2 "Package_LGA:Bosch_LGA-8_2.5x2.5mm_P0.65mm_ClockwisePinNumbering" H 4600 4600 50  0001 C CNN
-F 3 "https://ae-bst.resource.bosch.com/media/_tech/media/datasheets/BST-BME280_DS001-11.pdf" H 4600 4600 50  0001 C CNN
-	1    4600 4800
+P 7000 5300
+F 0 "U2" H 6570 5346 50  0000 R CNN
+F 1 "BME280" H 6570 5255 50  0000 R CNN
+F 2 "Package_LGA:Bosch_LGA-8_2.5x2.5mm_P0.65mm_ClockwisePinNumbering" H 7000 5100 50  0001 C CNN
+F 3 "https://ae-bst.resource.bosch.com/media/_tech/media/datasheets/BST-BME280_DS001-11.pdf" H 7000 5100 50  0001 C CNN
+	1    7000 5300
 	1    0    0    -1
 $EndComp
@@
 L Switch:SW_Push SW1
 U 1 1 5CA65465
-P 9150 1700
-F 0 "SW1" H 9150 1985 50  0000 C CNN
-F 1 "SW_Push" H 9150 1894 50  0000 C CNN
-F 2 "" H 9150 1900 50  0001 C CNN
-F 3 "" H 9150 1900 50  0001 C CNN
-	1    9150 1700
+P 5350 4150
+F 0 "SW1" H 5350 4435 50  0000 C CNN
+F 1 "SW_Push" H 5350 4344 50  0000 C CNN
+F 2 "" H 5350 4350 50  0001 C CNN
+F 3 "" H 5350 4350 50  0001 C CNN
+	1    5350 4150
 	1    0    0    -1
 $EndComp
@@
 L Switch:SW_Push SW2
 U 1 1 5CA6551B
-P 9150 2300
-F 0 "SW2" H 9150 2585 50  0000 C CNN
-F 1 "SW_Push" H 9150 2494 50  0000 C CNN
-F 2 "" H 9150 2500 50  0001 C CNN
-F 3 "" H 9150 2500 50  0001 C CNN
-	1    9150 2300
+P 3600 3500
+F 0 "SW2" H 3600 3785 50  0000 C CNN
+F 1 "SW_Push" H 3600 3694 50  0000 C CNN
+F 2 "" H 3600 3700 50  0001 C CNN
+F 3 "" H 3600 3700 50  0001 C CNN
+	1    3600 3500
 	1    0    0    -1
 $EndComp
@@
 $EndComp
 Wire Wire Line
-	5200 4900 5750 4900
-Wire Wire Line
 	5850 4900 5850 3300
 Wire Wire Line
 	5050 3300 5850 3300
 Wire Wire Line
-	5800 3400 5800 4500
-Wire Wire Line
-	5800 4500 5200 4500
-Wire Wire Line
 	5050 3400 5800 3400
 Wire Wire Line
@@
 	5050 3200 5900 3200
 Wire Wire Line
-	5800 4500 5800 5350
-Wire Wire Line
 	5800 5350 5900 5350
-Connection ~ 5800 4500
 Wire Wire Line
 	5750 4900 5750 5450
 Wire Wire Line
 	5750 5450 6000 5450
-Connection ~ 5750 4900
 Wire Wire Line
 	5750 4900 5850 4900
@@
 Wire Wire Line
 	5650 5550 5950 5550
-Connection ~ 5650 4700
-Wire Wire Line
-	5650 4700 5200 4700
 $Comp
 L Connector:Conn_01x06_Male MICRO_SD1
@@
 $EndComp
 Wire Wire Line
-	5400 6100 5900 6100
+	5400 6100 5550 6100
 Wire Wire Line
 	5900 6100 5900 5350
-Connection ~ 5900 5350
-Wire Wire Line
-	5900 5350 6100 5350
-Wire Wire Line
-	5400 6200 5950 6200
+Wire Wire Line
+	5400 6200 5550 6200
 Wire Wire Line
 	5950 6200 5950 5550
-Connection ~ 5950 5550
-Wire Wire Line
-	5950 5550 6100 5550
-Wire Wire Line
-	5400 6300 6000 6300
+Wire Wire Line
+	5400 6300 5550 6300
 Wire Wire Line
 	6000 6300 6000 5450
-Connection ~ 6000 5450
-Wire Wire Line
-	6000 5450 6100 5450
 $Comp
 L power:GND #PWR0106
@@
 	5400 6400 5550 6400
 Wire Wire Line
-	5550 6400 5550 6450
-Wire Wire Line
 	5450 5550 5450 5900
 Wire Wire Line
 	5450 5900 5400 5900
-Wire Wire Line
-	4700 5400 4700 6450
-Wire Wire Line
-	4700 6450 5550 6450
-Connection ~ 5550 6450
-Wire Wire Line
-	5550 6450 5550 6500
-Wire Wire Line
-	4500 5400 4500 6500
-Wire Wire Line
-	4500 6500 5550 6500
-Connection ~ 5550 6500
-Wire Wire Line
-	4900 4300 4800 4300
-Wire Wire Line
-	4800 4300 4800 4200
-Wire Wire Line
-	4800 4200 4700 4200
-Wire Wire Line
-	7300 3100 7450 3100
-Wire Wire Line
-	6900 4750 6900 4550
-$Comp
-L power:+3V3 #PWR0107
-U 1 1 5CA89BB7
-P 4900 4300
-F 0 "#PWR0107" H 4900 4150 50  0001 C CNN
-F 1 "+3V3" H 4915 4473 50  0000 C CNN
-F 2 "" H 4900 4300 50  0001 C CNN
-F 3 "" H 4900 4300 50  0001 C CNN
-	1    4900 4300
-	1    0    0    -1
-$EndComp
 $Comp
 L power:+3V3 #PWR0108
 U 1 1 5CA89CBB
-P 6900 4550
-F 0 "#PWR0108" H 6900 4400 50  0001 C CNN
-F 1 "+3V3" H 6915 4723 50  0000 C CNN
-F 2 "" H 6900 4550 50  0001 C CNN
-F 3 "" H 6900 4550 50  0001 C CNN
-	1    6900 4550
+P 8800 4450
+F 0 "#PWR0108" H 8800 4300 50  0001 C CNN
+F 1 "+3V3" H 8815 4623 50  0000 C CNN
+F 2 "" H 8800 4450 50  0001 C CNN
+F 3 "" H 8800 4450 50  0001 C CNN
+	1    8800 4450
 	1    0    0    -1
 $EndComp
@@
 	1    0    0    -1
 $EndComp
-Wire Wire Line
-	5550 6500 5550 6550
-Wire Wire Line
-	6800 6550 5550 6550
-Connection ~ 5550 6550
-Wire Wire Line
-	5550 6550 5550 6650
 $Comp
 L Interface_Expansion:MCP23S17_SS U3
@@
 	1    0    0    -1
 $EndComp
+Wire Wire Line
+	5050 3500 5600 3500
+Wire Wire Line
+	5600 3500 5600 4150
+Wire Wire Line
+	5600 4150 5550 4150
+$Comp
+L power:GND #PWR?
+U 1 1 5CA77F28
+P 5150 4150
+F 0 "#PWR?" H 5150 3900 50  0001 C CNN
+F 1 "GND" H 5155 3977 50  0000 C CNN
+F 2 "" H 5150 4150 50  0001 C CNN
+F 3 "" H 5150 4150 50  0001 C CNN
+	1    5150 4150
+	1    0    0    -1
+$EndComp
+Wire Wire Line
+	3800 3500 4550 3500
+$Comp
+L power:GND #PWR?
+U 1 1 5CA7A5D4
+P 3400 3500
+F 0 "#PWR?" H 3400 3250 50  0001 C CNN
+F 1 "GND" H 3405 3327 50  0000 C CNN
+F 2 "" H 3400 3500 50  0001 C CNN
+F 3 "" H 3400 3500 50  0001 C CNN
+	1    3400 3500
+	1    0    0    -1
+$EndComp
+$Comp
+L Connector:Conn_01x06_Female SPI_HEADER
+U 1 1 5CA7AA74
+P 5750 6100
+F 0 "SPI_HEADER" H 5777 6076 50  0000 L CNN
+F 1 "Conn_01x06_Female" H 5777 5985 50  0000 L CNN
+F 2 "" H 5750 6100 50  0001 C CNN
+F 3 "~" H 5750 6100 50  0001 C CNN
+	1    5750 6100
+	1    0    0    -1
+$EndComp
+Connection ~ 5550 6100
+Wire Wire Line
+	5550 6100 5900 6100
+Connection ~ 5550 6200
+Wire Wire Line
+	5550 6200 5950 6200
+Connection ~ 5550 6300
+Wire Wire Line
+	5550 6300 6000 6300
+Connection ~ 5550 6400
+Wire Wire Line
+	5550 5900 5450 5900
+Connection ~ 5450 5900
+Wire Wire Line
+	8000 3100 8000 4950
+Wire Wire Line
+	7300 3100 8000 3100
+Wire Wire Line
+	7950 3000 7950 5200
+Wire Wire Line
+	7950 5250 8000 5250
+Wire Wire Line
+	7300 3000 7950 3000
+$Comp
+L power:+3V3 #PWR?
+U 1 1 5CA917C5
+P 7100 4700
+F 0 "#PWR?" H 7100 4550 50  0001 C CNN
+F 1 "+3V3" H 7115 4873 50  0000 C CNN
+F 2 "" H 7100 4700 50  0001 C CNN
+F 3 "" H 7100 4700 50  0001 C CNN
+	1    7100 4700
+	1    0    0    -1
+$EndComp
+Wire Wire Line
+	7600 5200 7950 5200
+Connection ~ 7950 5200
+Wire Wire Line
+	7950 5200 7950 5250
+Wire Wire Line
+	7600 5400 7800 5400
+Wire Wire Line
+	7800 5400 7800 4950
+Wire Wire Line
+	7800 4950 8000 4950
+Connection ~ 8000 4950
+Wire Wire Line
+	8000 4950 8000 5050
+$Comp
+L power:GND #PWR?
+U 1 1 5CAAD4CB
+P 7700 6150
+F 0 "#PWR?" H 7700 5900 50  0001 C CNN
+F 1 "GND" H 7705 5977 50  0000 C CNN
+F 2 "" H 7700 6150 50  0001 C CNN
+F 3 "" H 7700 6150 50  0001 C CNN
+	1    7700 6150
+	1    0    0    -1
+$EndComp
+Wire Wire Line
+	7100 5900 7700 5900
+Wire Wire Line
+	7700 5900 7700 6100
+Wire Wire Line
+	6900 5900 7100 5900
+Connection ~ 7100 5900
+Wire Wire Line
+	8700 6250 7950 6250
+Wire Wire Line
+	7950 6250 7950 6100
+Wire Wire Line
+	7950 6100 7700 6100
+Connection ~ 7700 6100
+Wire Wire Line
+	7700 6100 7700 6150
+Wire Wire Line
+	5550 6400 5550 6650
+Wire Wire Line
+	5800 3400 5800 5350
 $EndSCHEMATC

Commit message: Add TFT Display connector
Parts:
- added J4: Conn_01x08, Connector_FFC-FPC:Hirose_FH12-50S-0.5SH_1x50-1MP_P0.50mm_Horizontal, symbol Connector_Generic:Conn_01x08
- J3: footprint (none) -> Connector_Audio:Jack_3.5mm_CUI_SJ1-3533NG_Horizontal
- MICRO_SD1: footprint (none) -> Connector_PinHeader_2.54mm:PinHeader_1x06_P2.54mm_Vertical
- SPI_HEADER1: renamed from SPI_HEADER; footprint (none) -> Connector_PinSocket_2.54mm:PinSocket_1x06_P2.54mm_Vertical
Connections:
- net +3V3: now also J4.2 (Pin_2)
- net GND: now also J4.1 (Pin_1)
- net PIN_18: now also J4.5 (Pin_5)
- net PIN_19: now also J4.4 (Pin_4)
- net PIN_23: now also J4.3 (Pin_3)
Changed lines of the file:
@@
 F 0 "J3" H 6580 1525 50  0000 C CNN
 F 1 "AudioJack3" H 6580 1434 50  0000 C CNN
-F 2 "" H 6600 1200 50  0001 C CNN
+F 2 "Connector_Audio:Jack_3.5mm_CUI_SJ1-3533NG_Horizontal" H 6600 1200 50  0001 C CNN
 F 3 "~" H 6600 1200 50  0001 C CNN
 	1    6600 1200
@@
 	5800 5350 5900 5350
 Wire Wire Line
-	5750 4900 5750 5450
+	5750 4900 5750 5150
 Wire Wire Line
 	5750 5450 6000 5450
@@
 	5750 4900 5850 4900
 Wire Wire Line
-	5650 4700 5650 5550
+	5650 4700 5650 5050
 Wire Wire Line
 	5650 5550 5950 5550
@@
 F 0 "MICRO_SD1" H 5306 6478 50  0000 C CNN
 F 1 "Conn_01x06_Male" H 5306 6387 50  0000 C CNN
-F 2 "" H 5200 6100 50  0001 C CNN
+F 2 "Connector_PinHeader_2.54mm:PinHeader_1x06_P2.54mm_Vertical" H 5200 6100 50  0001 C CNN
 F 3 "~" H 5200 6100 50  0001 C CNN
 	1    5200 6100
@@
 	5400 6400 5550 6400
 Wire Wire Line
-	5450 5550 5450 5900
+	5450 5550 5450 5600
 Wire Wire Line
 	5450 5900 5400 5900
@@
 	5600 4150 5550 4150
 $Comp
-L power:GND #PWR?
+L power:GND #PWR0107
 U 1 1 5CA77F28
 P 5150 4150
-F 0 "#PWR?" H 5150 3900 50  0001 C CNN
+F 0 "#PWR0107" H 5150 3900 50  0001 C CNN
 F 1 "GND" H 5155 3977 50  0000 C CNN
 F 2 "" H 5150 4150 50  0001 C CNN
@@
 	3800 3500 4550 3500
 $Comp
-L power:GND #PWR?
+L power:GND #PWR0110
 U 1 1 5CA7A5D4
 P 3400 3500
-F 0 "#PWR?" H 3400 3250 50  0001 C CNN
+F 0 "#PWR0110" H 3400 3250 50  0001 C CNN
 F 1 "GND" H 3405 3327 50  0000 C CNN
 F 2 "" H 3400 3500 50  0001 C CNN
@@
 $EndComp
 $Comp
-L Connector:Conn_01x06_Female SPI_HEADER
+L Connector:Conn_01x06_Female SPI_HEADER1
 U 1 1 5CA7AA74
 P 5750 6100
-F 0 "SPI_HEADER" H 5777 6076 50  0000 L CNN
+F 0 "SPI_HEADER1" H 5777 6076 50  0000 L CNN
 F 1 "Conn_01x06_Female" H 5777 5985 50  0000 L CNN
-F 2 "" H 5750 6100 50  0001 C CNN
+F 2 "Connector_PinSocket_2.54mm:PinSocket_1x06_P2.54mm_Vertical" H 5750 6100 50  0001 C CNN
 F 3 "~" H 5750 6100 50  0001 C CNN
 	1    5750 6100
@@
 	7300 3000 7950 3000
 $Comp
-L power:+3V3 #PWR?
+L power:+3V3 #PWR0111
 U 1 1 5CA917C5
 P 7100 4700
-F 0 "#PWR?" H 7100 4550 50  0001 C CNN
+F 0 "#PWR0111" H 7100 4550 50  0001 C CNN
 F 1 "+3V3" H 7115 4873 50  0000 C CNN
 F 2 "" H 7100 4700 50  0001 C CNN
@@
 	8000 4950 8000 5050
 $Comp
-L power:GND #PWR?
+L power:GND #PWR0112
 U 1 1 5CAAD4CB
 P 7700 6150
-F 0 "#PWR?" H 7700 5900 50  0001 C CNN
+F 0 "#PWR0112" H 7700 5900 50  0001 C CNN
 F 1 "GND" H 7705 5977 50  0000 C CNN
 F 2 "" H 7700 6150 50  0001 C CNN
@@
 	7700 6100 7700 6150
 Wire Wire Line
-	5550 6400 5550 6650
-Wire Wire Line
-	5800 3400 5800 5350
+	5550 6400 5550 6550
+$Comp
+L Connector_Generic:Conn_01x08 J4
+U 1 1 5CA73EBA
+P 4750 5150
+F 0 "J4" H 4670 4525 50  0000 C CNN
+F 1 "Conn_01x08" H 4670 4616 50  0000 C CNN
+F 2 "Connector_FFC-FPC:Hirose_FH12-50S-0.5SH_1x50-1MP_P0.50mm_Horizontal" H 4750 5150 50  0001 C CNN
+F 3 "~" H 4750 5150 50  0001 C CNN
+	1    4750 5150
+	-1   0    0    1
+$EndComp
+Wire Wire Line
+	4950 5050 5650 5050
+Connection ~ 5650 5050
+Wire Wire Line
+	5650 5050 5650 5550
+Wire Wire Line
+	4950 5150 5750 5150
+Connection ~ 5750 5150
+Wire Wire Line
+	5750 5150 5750 5450
+Wire Wire Line
+	4950 5250 5800 5250
+Wire Wire Line
+	5800 3400 5800 5250
+Connection ~ 5800 5250
+Wire Wire Line
+	5800 5250 5800 5350
+Wire Wire Line
+	4950 5350 5300 5350
+Wire Wire Line
+	5300 5350 5300 5600
+Wire Wire Line
+	5300 5600 5450 5600
+Connection ~ 5450 5600
+Wire Wire Line
+	5450 5600 5450 5900
+Wire Wire Line
+	4950 5450 4950 6550
+Wire Wire Line
+	4950 6550 5550 6550
+Connection ~ 5550 6550
+Wire Wire Line
+	5550 6550 5550 6650
 $EndSCHEMATC
