File: workshop_controller.sch (KiCad schematic (older format))
At the start: 47 parts, among them J1 Conn_02x10_Odd_Even, J2 Conn_02x10_Odd_Even, J3 AudioJack3, J4 Micro_SD_Card, J5 Conn_02x25_Odd_Even, M1 Microphone4, SW1 SW_Push, SW2 SW_Push, SW3 SW_Push, SW4 SW_Push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

Commit message: Add 2020 led
Parts:
- removed JOYSTICK_LEFT1: R_POT_Dual, symbol Device:R_POT_Dual
- added D1: LED_RGB, LED_SMD:LED_ROHM_SMLVN6, symbol Device:LED_RGB
- added D2: APA102, GSG:APA102-2020, symbol GSG:APA102
- added U6: PSP_1000_JSTK, HackPack4:JOYSTICK-PSP1000, symbol HackPack4:HackPackv4-rescue_PSP_1000_JSTK
Other:
- moved on the sheet: SW1, SW2, SW3, SW4
Changed lines of the file:
@@
 L Switch:SW_Push SW1
 U 1 1 5CA65465
-P 2150 2800
-F 0 "SW1" H 2150 3085 50  0000 C CNN
-F 1 "SW_Push" H 2150 2994 50  0000 C CNN
-F 2 "Button_Switch_THT:SW_PUSH-12mm_Wuerth-430476085716" H 2150 3000 50  0001 C CNN
-F 3 "" H 2150 3000 50  0001 C CNN
-	1    2150 2800
+P 1000 2900
+F 0 "SW1" H 1000 3185 50  0000 C CNN
+F 1 "SW_Push" H 1000 3094 50  0000 C CNN
+F 2 "Button_Switch_THT:SW_PUSH-12mm_Wuerth-430476085716" H 1000 3100 50  0001 C CNN
+F 3 "" H 1000 3100 50  0001 C CNN
+	1    1000 2900
 	1    0    0    -1
 $EndComp
@@
 L Switch:SW_Push SW2
 U 1 1 5CA6551B
-P 2150 3150
-F 0 "SW2" H 2150 3435 50  0000 C CNN
-F 1 "SW_Push" H 2150 3344 50  0000 C CNN
-F 2 "Button_Switch_THT:SW_PUSH-12mm_Wuerth-430476085716" H 2150 3350 50  0001 C CNN
-F 3 "" H 2150 3350 50  0001 C CNN
-	1    2150 3150
+P 1000 3250
+F 0 "SW2" H 1000 3535 50  0000 C CNN
+F 1 "SW_Push" H 1000 3444 50  0000 C CNN
+F 2 "Button_Switch_THT:SW_PUSH-12mm_Wuerth-430476085716" H 1000 3450 50  0001 C CNN
+F 3 "" H 1000 3450 50  0001 C CNN
+	1    1000 3250
 	1    0    0    -1
 $EndComp
@@
 F 3 "~" H 4000 1200 50  0001 C CNN
 	1    4000 1200
-	1    0    0    -1
-$EndComp
-$Comp
-L Device:R_POT_Dual JOYSTICK_LEFT1
-U 1 1 5CA65DAB
-P 4150 1950
-F 0 "JOYSTICK_LEFT1" H 4150 1718 50  0000 C CNN
-F 1 "R_POT_Dual" H 4150 1627 50  0000 C CNN
-F 2 "" H 4400 1875 50  0001 C CNN
-F 3 "~" H 4400 1875 50  0001 C CNN
-	1    4150 1950
 	1    0    0    -1
 $EndComp
@@
 L Switch:SW_Push SW3
 U 1 1 5CC6CBA8
-P 2150 3500
-F 0 "SW3" H 2150 3785 50  0000 C CNN
-F 1 "SW_Push" H 2150 3694 50  0000 C CNN
-F 2 "Button_Switch_THT:SW_PUSH-12mm_Wuerth-430476085716" H 2150 3700 50  0001 C CNN
-F 3 "~" H 2150 3700 50  0001 C CNN
-	1    2150 3500
+P 1000 3600
+F 0 "SW3" H 1000 3885 50  0000 C CNN
+F 1 "SW_Push" H 1000 3794 50  0000 C CNN
+F 2 "Button_Switch_THT:SW_PUSH-12mm_Wuerth-430476085716" H 1000 3800 50  0001 C CNN
+F 3 "~" H 1000 3800 50  0001 C CNN
+	1    1000 3600
 	1    0    0    -1
 $EndComp
@@
 L Switch:SW_Push SW4
 U 1 1 5CC6E62A
-P 2150 3850
-F 0 "SW4" H 2150 4135 50  0000 C CNN
-F 1 "SW_Push" H 2150 4044 50  0000 C CNN
-F 2 "Button_Switch_THT:SW_PUSH-12mm_Wuerth-430476085716" H 2150 4050 50  0001 C CNN
-F 3 "~" H 2150 4050 50  0001 C CNN
-	1    2150 3850
+P 1000 3950
+F 0 "SW4" H 1000 4235 50  0000 C CNN
+F 1 "SW_Push" H 1000 4144 50  0000 C CNN
+F 2 "Button_Switch_THT:SW_PUSH-12mm_Wuerth-430476085716" H 1000 4150 50  0001 C CNN
+F 3 "~" H 1000 4150 50  0001 C CNN
+	1    1000 3950
 	1    0    0    -1
 $EndComp
@@
 L power:GND #PWR0132
 U 1 1 5CC6F72D
-P 1950 2800
-F 0 "#PWR0132" H 1950 2550 50  0001 C CNN
-F 1 "GND" V 1955 2672 50  0000 R CNN
-F 2 "" H 1950 2800 50  0001 C CNN
-F 3 "" H 1950 2800 50  0001 C CNN
-	1    1950 2800
+P 800 2900
+F 0 "#PWR0132" H 800 2650 50  0001 C CNN
+F 1 "GND" V 805 2772 50  0000 R CNN
+F 2 "" H 800 2900 50  0001 C CNN
+F 3 "" H 800 2900 50  0001 C CNN
+	1    800  2900
 	0    1    1    0
 $EndComp
@@
 L power:GND #PWR0133
 U 1 1 5CC70236
-P 1950 3150
-F 0 "#PWR0133" H 1950 2900 50  0001 C CNN
-F 1 "GND" V 1955 3022 50  0000 R CNN
-F 2 "" H 1950 3150 50  0001 C CNN
-F 3 "" H 1950 3150 50  0001 C CNN
-	1    1950 3150
+P 800 3250
+F 0 "#PWR0133" H 800 3000 50  0001 C CNN
+F 1 "GND" V 805 3122 50  0000 R CNN
+F 2 "" H 800 3250 50  0001 C CNN
+F 3 "" H 800 3250 50  0001 C CNN
+	1    800  3250
 	0    1    1    0
 $EndComp
@@
 L power:GND #PWR0134
 U 1 1 5CC70C86
-P 1950 3500
-F 0 "#PWR0134" H 1950 3250 50  0001 C CNN
-F 1 "GND" V 1955 3372 50  0000 R CNN
-F 2 "" H 1950 3500 50  0001 C CNN
-F 3 "" H 1950 3500 50  0001 C CNN
-	1    1950 3500
+P 800 3600
+F 0 "#PWR0134" H 800 3350 50  0001 C CNN
+F 1 "GND" V 805 3472 50  0000 R CNN
+F 2 "" H 800 3600 50  0001 C CNN
+F 3 "" H 800 3600 50  0001 C CNN
+	1    800  3600
 	0    1    1    0
 $EndComp
@@
 L power:GND #PWR0135
 U 1 1 5CC7168C
-P 1950 3850
-F 0 "#PWR0135" H 1950 3600 50  0001 C CNN
-F 1 "GND" V 1955 3722 50  0000 R CNN
-F 2 "" H 1950 3850 50  0001 C CNN
-F 3 "" H 1950 3850 50  0001 C CNN
-	1    1950 3850
-	0    1    1    0
-$EndComp
-Text Label 2350 2800 0    50   ~ 0
+P 800 3950
+F 0 "#PWR0135" H 800 3700 50  0001 C CNN
+F 1 "GND" V 805 3822 50  0000 R CNN
+F 2 "" H 800 3950 50  0001 C CNN
+F 3 "" H 800 3950 50  0001 C CNN
+	1    800  3950
+	0    1    1    0
+$EndComp
+Text Label 1200 2900 0    50   ~ 0
 SW1_PIN
-Text Label 2350 3150 0    50   ~ 0
+Text Label 1200 3250 0    50   ~ 0
 SW2_PIN
-Text Label 2350 3500 0    50   ~ 0
+Text Label 1200 3600 0    50   ~ 0
 SW3_PIN
-Text Label 2350 3850 0    50   ~ 0
+Text Label 1200 3950 0    50   ~ 0
 SW4_PIN
 Text Label 5550 3500 0    50   ~ 0
@@
 Wire Wire Line
 	4000 3400 4550 3400
-Text Label 3900 1850 2    50   ~ 0
-JOY_X
-Text Label 4400 1850 0    50   ~ 0
-JOY_Y
-$Comp
-L power:GND #PWR0138
-U 1 1 5CD0AC46
-P 4050 2050
-F 0 "#PWR0138" H 4050 1800 50  0001 C CNN
-F 1 "GND" H 4055 1877 50  0000 C CNN
-F 2 "" H 4050 2050 50  0001 C CNN
-F 3 "" H 4050 2050 50  0001 C CNN
-	1    4050 2050
-	1    0    0    -1
-$EndComp
-$Comp
-L power:GND #PWR0139
-U 1 1 5CD0AFBD
-P 4550 2050
-F 0 "#PWR0139" H 4550 1800 50  0001 C CNN
-F 1 "GND" H 4555 1877 50  0000 C CNN
-F 2 "" H 4550 2050 50  0001 C CNN
-F 3 "" H 4550 2050 50  0001 C CNN
-	1    4550 2050
-	1    0    0    -1
-$EndComp
-$Comp
-L power:+3V3 #PWR0140
-U 1 1 5CD0C0CF
-P 3750 2050
-F 0 "#PWR0140" H 3750 1900 50  0001 C CNN
-F 1 "+3V3" H 3765 2223 50  0000 C CNN
-F 2 "" H 3750 2050 50  0001 C CNN
-F 3 "" H 3750 2050 50  0001 C CNN
-	1    3750 2050
-	-1   0    0    1
-$EndComp
-$Comp
-L power:+3V3 #PWR0141
-U 1 1 5CD0D40E
-P 4250 2050
-F 0 "#PWR0141" H 4250 1900 50  0001 C CNN
-F 1 "+3V3" H 4265 2223 50  0000 C CNN
-F 2 "" H 4250 2050 50  0001 C CNN
-F 3 "" H 4250 2050 50  0001 C CNN
-	1    4250 2050
-	-1   0    0    1
-$EndComp
 $Comp
 L bytebarista:Microphone4 M1
@@
 PIN_DAC2
 $Comp
-L power:GND #PWR?
+L power:GND #PWR0156
 U 1 1 5CBFD31D
 P 9750 3450
-F 0 "#PWR?" H 9750 3200 50  0001 C CNN
+F 0 "#PWR0156" H 9750 3200 50  0001 C CNN
 F 1 "GND" H 9755 3277 50  0000 C CNN
 F 2 "" H 9750 3450 50  0001 C CNN
@@
 	1    0    0    -1
 $EndComp
+$Comp
+L Device:LED_RGB D1
+U 1 1 5CC0060A
+P 5000 4750
+F 0 "D1" H 5000 5247 50  0000 C CNN
+F 1 "LED_RGB" H 5000 5156 50  0000 C CNN
+F 2 "LED_SMD:LED_ROHM_SMLVN6" H 5000 4700 50  0001 C CNN
+F 3 "~" H 5000 4700 50  0001 C CNN
+	1    5000 4750
+	1    0    0    -1
+$EndComp
+$Comp
+L GSG:APA102 D2
+U 1 1 5CBA7953
+P 5950 2350
+F 0 "D2" H 5950 2787 60  0000 C CNN
+F 1 "APA102" H 5950 2681 60  0000 C CNN
+F 2 "GSG:APA102-2020" H 5950 2350 60  0001 C CNN
+F 3 "" H 5950 2350 60  0001 C CNN
+	1    5950 2350
+	1    0    0    -1
+$EndComp
+$Comp
+L power:GND #PWR0157
+U 1 1 5CBA7A63
+P 5600 2450
+F 0 "#PWR0157" H 5600 2200 50  0001 C CNN
+F 1 "GND" H 5605 2277 50  0000 C CNN
+F 2 "" H 5600 2450 50  0001 C CNN
+F 3 "" H 5600 2450 50  0001 C CNN
+	1    5600 2450
+	1    0    0    -1
+$EndComp
+$Comp
+L power:+3V3 #PWR0158
+U 1 1 5CBA7B5D
+P 6300 2450
+F 0 "#PWR0158" H 6300 2300 50  0001 C CNN
+F 1 "+3V3" H 6315 2623 50  0000 C CNN
+F 2 "" H 6300 2450 50  0001 C CNN
+F 3 "" H 6300 2450 50  0001 C CNN
+	1    6300 2450
+	-1   0    0    1
+$EndComp
+$Comp
+L HackPack4:HackPackv4-rescue_PSP_1000_JSTK U6
+U 1 1 5CBA7E0F
+P 2400 3050
+F 0 "U6" H 2727 3053 60  0000 L CNN
+F 1 "PSP_1000_JSTK" H 2727 2947 60  0000 L CNN
+F 2 "HackPack4:JOYSTICK-PSP1000" H 3700 2350 60  0001 C CNN
+F 3 "" H 3700 2350 60  0001 C CNN
+	1    2400 3050
+	1    0    0    -1
+$EndComp
+$Comp
+L power:GND #PWR0159
+U 1 1 5CBA7FD8
+P 2400 3800
+F 0 "#PWR0159" H 2400 3550 50  0001 C CNN
+F 1 "GND" H 2405 3627 50  0000 C CNN
+F 2 "" H 2400 3800 50  0001 C CNN
+F 3 "" H 2400 3800 50  0001 C CNN
+	1    2400 3800
+	1    0    0    -1
+$EndComp
+$Comp
+L power:+3V3 #PWR0160
+U 1 1 5CBA80D5
+P 2400 2400
+F 0 "#PWR0160" H 2400 2250 50  0001 C CNN
+F 1 "+3V3" H 2415 2573 50  0000 C CNN
+F 2 "" H 2400 2400 50  0001 C CNN
+F 3 "" H 2400 2400 50  0001 C CNN
+	1    2400 2400
+	1    0    0    -1
+$EndComp
+Text Label 1900 3000 2    50   ~ 0
+JOY_X
+Text Label 1900 3100 2    50   ~ 0
+JOY_Y
 $EndSCHEMATC

Commit message: Add tracks for prototype^C
Parts:
- removed D1: LED_RGB, LED_SMD:LED_ROHM_SMLVN6, symbol Device:LED_RGB
- added D1, D3, D4: APA102, GSG:APA102-2020, symbol GSG:APA102
- added J6: Conn_01x05_Female, Connector_PinHeader_2.54mm:PinHeader_1x05_P2.54mm_Horizontal, symbol Connector:Conn_01x05_Female
- added J7: LOGO_TOUCH, Hackheim_logo:F.Cu_g9870, symbol Connector:Conn_01x01_Male
Connections:
- net labels added: GPIO_EXT_1, GPIO_EXT_2, GPIO_EXT_3, LED_CLK, LED_DA, PIN_LOGO_TOUCH, PIN_RESET_TFT, SPI_SCL, SPI_SDI, SPI_SDO
- net labels removed: PIN_RESET, PIN_SCL, PIN_SDI, SPEAKER
Other:
- moved on the sheet: I2C_HEADER1, J5
